File: modular_ad74416h_plc/modular_ad74416h_plc.kicad_pcb (KiCad board)
At the start: 2 copper layers, 5.1 x 5.1 mm, 0 parts

Commit message: Backup: Updated KiCad project files and submodule
Parts:
- added MOD1: ~, modules_footprints:ad74416h_power_interface_module, F.Cu at (156.5, 100.8)
Changed lines of the file:
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@@
 	)
 	(net 0 "")
+	(footprint "modules_footprints:ad74416h_power_interface_module"
+		(layer "F.Cu")
+		(at 156.4894 100.7618)
+		(property "Reference" "MOD1"
+			(at 0 -0.5 0)
+			(unlocked yes)
+			(layer "F.SilkS")
+			(effects
+				(font
+					(size 1 1)
+					(thickness 0.1)
+				)
+			)
+		)
+		(property "Value" "~"
+			(at 0 1 0)
+			(unlocked yes)
+			(layer "F.Fab")
+			(effects
+				(font
+					(size 1 1)
+					(thickness 0.15)
+				)
+			)
+		)
+		(property "Datasheet" ""
+			(at 0 0 0)
+			(unlocked yes)
+			(layer "F.Fab")
+			(hide yes)
+			(effects
+				(font
+					(size 1 1)
+					(thickness 0.15)
+				)
+			)
+		)
+		(property "Description" ""
+			(at 0 0 0)
+			(unlocked yes)
+			(layer "F.Fab")
+			(hide yes)
+			(effects
+				(font
+					(size 1 1)
+					(thickness 0.15)
+				)
+			)
+		)
+		(sheetname "/")
+		(sheetfile "modular_ad74416h_plc.kicad_sch")
+		(fp_text user "${REFERENCE}"
+			(at 0 2.5 0)
+			(unlocked yes)
+			(layer "F.Fab")
+			(effects
+				(font
+					(size 1 1)
+					(thickness 0.15)
+				)
+			)
+		)
+		(embedded_fonts no)
+		(model "${KICAD9_3D_MODELS_VAULT}/3D_models/modules/ad74416h_power_interface_module.step"
+			(offset
+				(xyz 0 0 -4)
+			)
+			(scale
+				(xyz 1 1 1)
+			)
+			(rotate
+				(xyz -0 -0 -0)
+			)
+		)
+	)
 	(gr_rect
 		(start 153.9494 98.2218)

Commit message: backup
Parts:
- added U1: ~, modules_footprints:minimal_ad74416h, F.Cu at (143.0, 84.4)
- added U2: ~, modules_footprints:minimal_ad74416h, F.Cu at (143.0, 79.3)
- added U3: ~, modules_footprints:minimal_ad74416h, F.Cu at (143.0, 74.1)
- added U4: ~, modules_footprints:minimal_ad74416h, F.Cu at (143.0, 68.9)
- moved MOD1 28.9 mm to (143.0, 126.4)
Other:
- board size 5.1 x 5.1 mm -> 54.4 x 46.3 mm

Commit message: backup
Parts:
- moved MOD1 5.84 mm to (143.0, 132.2)

Commit message: backup
Other:
- board size 54.4 x 46.3 mm -> 45.7 x 38.1 mm
Changed lines of the file:
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@@
 	(generator_version "9.0")
 	(general
-		(thickness 1.6)
+		(thickness 1.092)
 		(legacy_teardrops no)
 	)
@@
 	)
 	(setup
+		(stackup
+			(layer "F.SilkS"
+				(type "Top Silk Screen")
+			)
+			(layer "F.Paste"
+				(type "Top Solder Paste")
+			)
+			(layer "F.Mask"
+				(type "Top Solder Mask")
+				(thickness 0.01)
+			)
+			(layer "F.Cu"
+				(type "copper")
+				(thickness 0.035)
+			)
+			(layer "dielectric 1"
+				(type "core")
+				(thickness 1.002)
+				(material "FR4")
+				(epsilon_r 4.5)
+				(loss_tangent 0.02)
+			)
+			(layer "B.Cu"
+				(type "copper")
+				(thickness 0.035)
+			)
+			(layer "B.Mask"
+				(type "Bottom Solder Mask")
+				(thickness 0.01)
+			)
+			(layer "B.Paste"
+				(type "Bottom Solder Paste")
+			)
+			(layer "B.SilkS"
+				(type "Bottom Silk Screen")
+			)
+			(copper_finish "None")
+			(dielectric_constraints no)
+		)
 		(pad_to_mask_clearance 0)
 		(allow_soldermask_bridges_in_footprints no)
@@
 		(model "${KICAD9_3D_MODELS_VAULT}/3D_models/modules/minimal_ad74416h.step"
 			(offset
-				(xyz 0 0 11.43)
+				(xyz 0 0 10.16)
 			)
 			(scale
@@
 		(model "${KICAD9_3D_MODELS_VAULT}/3D_models/modules/ad74416h_power_interface_module.step"
 			(offset
-				(xyz 0 0 -4)
+				(xyz 0 0 -5.270000001)
 			)
 			(scale
@@
 		(model "${KICAD9_3D_MODELS_VAULT}/3D_models/modules/minimal_ad74416h.step"
 			(offset
-				(xyz 0 0 34.29)
+				(xyz 0 0 33.02)
 			)
 			(scale
@@
 		(model "${KICAD9_3D_MODELS_VAULT}/3D_models/modules/minimal_ad74416h.step"
 			(offset
-				(xyz 0 0 0)
+				(xyz 0 0 -1.27)
 			)
 			(scale
@@
 			)
 			(rotate
-				(xyz 0 0 0)
+				(xyz -0 -0 -0)
 			)
 		)
@@
 		(model "${KICAD9_3D_MODELS_VAULT}/3D_models/modules/minimal_ad74416h.step"
 			(offset
-				(xyz 0 0 22.86)
+				(xyz 0 0 21.59)
 			)
 			(scale
@@
 		)
 	)
-	(gr_rect
-		(start 116.205 54.5338)
-		(end 170.6372 100.838)
+	(gr_arc
+		(start 120.1547 59.7662)
+		(mid 120.377885 59.227385)
+		(end 120.9167 59.0042)
+		(stroke
+			(width 0.05)
+			(type default)
+		)
+		(layer "Edge.Cuts")
+	)
+	(gr_line
+		(start 120.1547 96.3422)
+		(end 120.1547 59.7662)
+		(stroke
+			(width 0.05)
+			(type default)
+		)
+		(layer "Edge.Cuts")
+	)
+	(gr_line
+		(start 120.9167 59.0042)
+		(end 165.1381 59.0042)
+		(stroke
+			(width 0.05)
+			(type default)
+		)
+		(layer "Edge.Cuts")
+	)
+	(gr_arc
+		(start 165.9001 96.3422)
+		(mid 165.676915 96.881015)
+		(end 165.1381 97.1042)
+		(stroke
+			(width 0.05)
+			(type default)
+		)
+		(layer "Edge.Cuts")
+	)
+	(gr_arc
+		(start 165.1381 59.0042)
+		(mid 165.676915 59.227385)
+		(end 165.9001 59.7662)
+		(stroke
+			(width 0.05)
+			(type default)
+		)
+		(layer "Edge.Cuts")
+	)
+	(gr_line
+		(start 165.1381 97.1042)
+		(end 120.9167 97.1042)
+		(stroke
+			(width 0.05)
+			(type default)
+		)
+		(layer "Edge.Cuts")
+	)
+	(gr_arc
+		(start 120.9167 97.1042)
+		(mid 120.377885 96.881015)
+		(end 120.1547 96.3422)
+		(stroke
+			(width 0.05)
+			(type default)
+		)
+		(layer "Edge.Cuts")
+	)
+	(gr_line
+		(start 165.9001 59.7662)
+		(end 165.9001 96.3422)
 		(stroke
 			(width 0.05)
-			(type solid)
+			(type default)
 		)
-		(fill no)
 		(layer "Edge.Cuts")
 	)

Commit message: backup
Other:
- board size 45.7 x 38.1 mm -> 45.7 x 2.5 mm
Changed lines of the file:
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@@
 	)
 	(gr_arc
-		(start 120.1547 59.7662)
-		(mid 120.377885 59.227385)
-		(end 120.9167 59.0042)
+		(start 120.1547 97.9424)
+		(mid 120.377885 97.403585)
+		(end 120.9167 97.1804)
 		(stroke
 			(width 0.05)
@@
 	)
 	(gr_line
-		(start 120.1547 96.3422)
-		(end 120.1547 59.7662)
+		(start 120.1547 98.9584)
+		(end 120.1547 97.9424)
+		(stroke
+			(width 0.05)
+			(type solid)
+		)
+		(layer "Edge.Cuts")
+	)
+	(gr_line
+		(start 120.9167 97.1804)
+		(end 165.1381 97.1804)
+		(stroke
+			(width 0.05)
+			(type default)
+		)
+		(layer "Edge.Cuts")
+	)
+	(gr_arc
+		(start 165.9001 98.9584)
+		(mid 165.676915 99.497215)
+		(end 165.1381 99.7204)
+		(stroke
+			(width 0.05)
+			(type default)
+		)
+		(layer "Edge.Cuts")
+	)
+	(gr_arc
+		(start 165.1381 97.1804)
+		(mid 165.676915 97.403585)
+		(end 165.9001 97.9424)
 		(stroke
 			(width 0.05)
@@
 	)
 	(gr_line
-		(start 120.9167 59.0042)
-		(end 165.1381 59.0042)
+		(start 165.1381 99.7204)
+		(end 120.9167 99.7204)
 		(stroke
 			(width 0.05)
@@
 	)
 	(gr_arc
-		(start 165.9001 96.3422)
-		(mid 165.676915 96.881015)
-		(end 165.1381 97.1042)
-		(stroke
-			(width 0.05)
-			(type default)
-		)
-		(layer "Edge.Cuts")
-	)
-	(gr_arc
-		(start 165.1381 59.0042)
-		(mid 165.676915 59.227385)
-		(end 165.9001 59.7662)
+		(start 120.9167 99.7204)
+		(mid 120.377885 99.497215)
+		(end 120.1547 98.9584)
 		(stroke
 			(width 0.05)
@@
 	)
 	(gr_line
-		(start 165.1381 97.1042)
-		(end 120.9167 97.1042)
+		(start 165.9001 97.9424)
+		(end 165.9001 98.9584)
 		(stroke
 			(width 0.05)
-			(type default)
+			(type solid)
 		)
 		(layer "Edge.Cuts")
-	)
-	(gr_arc
-		(start 120.9167 97.1042)
-		(mid 120.377885 96.881015)
-		(end 120.1547 96.3422)
-		(stroke
-			(width 0.05)
-			(type default)
-		)
-		(layer "Edge.Cuts")
-	)
-	(gr_line
-		(start 165.9001 59.7662)
-		(end 165.9001 96.3422)
-		(stroke
-			(width 0.05)
-			(type default)
-		)
-		(layer "Edge.Cuts")

Commit message: backup
Parts:
- moved MOD1 1.08 mm to (143.0, 131.2)
