File: modular_ad74416h_plc/modular_ad74416h_plc.kicad_pcb (KiCad board)
At the start: 2 copper layers, 45.7 x 2.5 mm, 7 parts

Commit message: backup
Parts:
- moved U3 0.10 mm to (193.8, 113.7)
- moved U4 0.10 mm to (193.8, 95.9)
Changed lines of the file:
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@@
 		(model "${KICAD9_3D_MODELS_VAULT}/3D_models/modules/minimal_ad74416h.step"
 			(offset
-				(xyz 0 0 6.985)
+				(xyz 0 0 4.318)
 			)
 			(scale
@@
 	(footprint "modules_footprints:minimal_ad74416h"
 		(layer "F.Cu")
-		(at 193.8274 96.012)
+		(at 193.8274 95.90786)
 		(property "Reference" "U4"
 			(at 0 -0.5 0)
@@
 		(model "${KICAD9_3D_MODELS_VAULT}/3D_models/modules/minimal_ad74416h.step"
 			(offset
-				(xyz 0 0 23.495)
+				(xyz 0 0 15.748)
 			)
 			(scale
@@
 	(footprint "modules_footprints:minimal_ad74416h"
 		(layer "F.Cu")
-		(at 193.8274 113.792)
+		(at 193.8274 113.68786)
 		(property "Reference" "U3"
 			(at 0 -0.5 0)
@@
 		(model "${KICAD9_3D_MODELS_VAULT}/3D_models/modules/minimal_ad74416h.step"
 			(offset
-				(xyz 0 0 15.24)
+				(xyz 0 0 10.033)
 			)
 			(scale
@@
 	(footprint "modules_footprints:minimal_adpl76030"
 		(layer "F.Cu")
-		(at 210.3501 207.2259 -90)
+		(at 210.3374 207.2259 -90)
 		(property "Reference" "U5"
 			(at 0 0 270)

Commit message: backup
Parts:
- moved U4 26.7 mm to (193.8, 122.6)
- moved U3 26.7 mm to (193.8, 140.4)
- moved U1 8.89 mm to (193.8, 140.4)
- moved U2 8.89 mm to (193.8, 122.6)

Commit message: backup
Parts:
- moved MOD2 1.27 mm to (193.8, 208.9)
- moved U5 1.27 mm to (210.3, 208.5)

Commit message: backup
Parts:
- moved MOD2 1.27 mm to (193.8, 210.2)
- moved U5 1.27 mm to (210.3, 209.8)

Commit message: backup
Parts:
- moved MOD2 5.08 mm to (193.8, 215.3)
- moved U5 5.08 mm to (210.3, 214.8)
- moved MOD1 2.54 mm to (193.8, 210.8)

Commit message: backup
Parts:
- moved U2 17.8 mm to (193.8, 140.4)
- moved U4 17.8 mm to (193.8, 140.4)
- moved MOD1 9.27 mm to (193.8, 201.6)
- moved MOD2 9.27 mm to (193.8, 206.0)
- moved U5 9.27 mm to (210.3, 205.6)

Commit message: backup
Parts:
- moved MOD1 15.4 mm to (193.8, 186.2)
- moved MOD2 15.4 mm to (193.8, 190.6)
- moved U1 15.4 mm to (193.8, 125.0)
- moved U2 15.4 mm to (193.8, 125.0)
- moved U3 15.4 mm to (193.8, 125.0)
- moved U4 15.4 mm to (193.8, 125.0)
- moved U5 15.4 mm to (210.3, 190.2)
Changed lines of the file:
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@@
 	(footprint "modules_footprints:minimal_adp1074"
 		(layer "F.Cu")
-		(at 193.8274 206.0194)
+		(at 193.8274 190.64986)
 		(property "Reference" "MOD2"
 			(at 0 0 0)
@@
 	(footprint "modules_footprints:minimal_ad74416h"
 		(layer "F.Cu")
-		(at 193.8274 140.3604)
+		(at 193.8274 124.99086)
 		(property "Reference" "U2"
 			(at 0 -0.5 0)
@@
 	(footprint "modules_footprints:ad74416h_power_interface_module"
 		(layer "F.Cu")
-		(at 193.8274 201.5744)
+		(at 193.8274 186.20486)
 		(property "Reference" "MOD1"
 			(at 0 -0.5 0)
@@
 	(footprint "modules_footprints:minimal_ad74416h"
 		(layer "F.Cu")
-		(at 193.8274 140.3604)
+		(at 193.8274 124.99086)
 		(property "Reference" "U4"
 			(at 0 -0.5 0)
@@
 	(footprint "modules_footprints:minimal_ad74416h"
 		(layer "F.Cu")
-		(at 193.8274 140.3604)
+		(at 193.8274 124.99086)
 		(property "Reference" "U1"
 			(at 0 -0.5 0)
@@
 	(footprint "modules_footprints:minimal_ad74416h"
 		(layer "F.Cu")
-		(at 193.8274 140.3604)
+		(at 193.8274 124.99086)
 		(property "Reference" "U3"
 			(at 0 -0.5 0)
@@
 	(footprint "modules_footprints:minimal_adpl76030"
 		(layer "F.Cu")
-		(at 210.3374 205.5749 -90)
+		(at 210.3374 190.20536 -90)
 		(property "Reference" "U5"
 			(at 0 0 270)
@@
 			(type default)
 		)
+		(locked yes)
 		(layer "Edge.Cuts")
 	)
@@
 			(type solid)
 		)
+		(locked yes)
 		(layer "Edge.Cuts")
 	)
@@
 			(type default)
 		)
+		(locked yes)
 		(layer "Edge.Cuts")
 	)
@@
 			(type default)
 		)
+		(locked yes)
 		(layer "Edge.Cuts")
 	)
@@
 			(type default)
 		)
+		(locked yes)
 		(layer "Edge.Cuts")
 	)
@@
 			(type default)
 		)
+		(locked yes)
 		(layer "Edge.Cuts")
 	)
@@
 			(type default)
 		)
+		(locked yes)
 		(layer "Edge.Cuts")
 	)
@@
 			(type solid)
 		)
+		(locked yes)
 		(layer "Edge.Cuts")
 	)

Commit message: backup
Parts:
- moved U5 3.56 mm to (210.3, 186.6)
- moved MOD2 3.56 mm to (193.8, 187.1)
- moved MOD1 1.65 mm to (193.8, 184.6)
