File: modular_ad74416h_plc/modular_ad74416h_plc.kicad_sch (KiCad schematic)
At the start: 0 parts

Commit message: Backup: Updated KiCad project files and submodule
Parts:
- added MOD1: ~, modules_footprints:ad74416h_power_interface_module, symbol UNITED_MODULES_DATA_BASE:AD74416H_POWER_INTERFACE_MODULE
Changed lines of the file:
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@@
 	(generator_version "9.0")
 	(paper "A4")
+	(symbol
+		(lib_id "UNITED_MODULES_DATA_BASE:AD74416H_POWER_INTERFACE_MODULE")
+		(at 152.4 101.6 0)
+		(unit 1)
+		(exclude_from_sim no)
+		(in_bom yes)
+		(on_board yes)
+		(dnp no)
+		(fields_autoplaced yes)
+		(property "Reference" "MOD1"
+			(at 158.75 100.3299 0)
+			(effects
+				(font
+					(size 1.27 1.27)
+				)
+				(justify left)
+			)
+		)
+		(property "Value" "~"
+			(at 158.75 102.8699 0)
+			(effects
+				(font
+					(size 1.27 1.27)
+				)
+				(justify left)
+			)
+		)
+		(property "Footprint" "modules_footprints:ad74416h_power_interface_module"
+			(at 152.4 109.22 0)
+			(effects
+				(font
+					(size 1.27 1.27)
+				)
+				(justify left)
+				(hide yes)
+			)
+		)
+		(property "Datasheet" ""
+			(at 152.4 101.6 0)
+			(effects
+				(font
+					(size 1.27 1.27)
+				)
+				(hide yes)
+			)
+		)
+		(property "Description" ""
+			(at 152.4 101.6 0)
+			(effects
+				(font
+					(size 1.27 1.27)
+				)
+				(hide yes)
+			)
+		)
+		(instances
+			(project ""
+				(path "/947a17bd-6931-4ad8-bf27-70104debc844"
+					(reference "MOD1")
+					(unit 1)
+				)
+			)
+		)
+	)
 	(sheet_instances
 		(path "/"

Commit message: backup
Parts:
- added U1: ~, modules_footprints:minimal_ad74416h, symbol UNITED_MODULES_DATA_BASE:MINIMAL_AD74416H
Changed lines of the file:
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@@
 	(paper "A4")
+	(symbol
+		(lib_id "UNITED_MODULES_DATA_BASE:MINIMAL_AD74416H")
+		(at 177.8 101.6 0)
+		(unit 1)
+		(exclude_from_sim no)
+		(in_bom yes)
+		(on_board yes)
+		(dnp no)
+		(fields_autoplaced yes)
+		(property "Reference" "U1"
+			(at 184.15 100.3299 0)
+			(effects
+				(font
+					(size 1.27 1.27)
+				)
+				(justify left)
+			)
+		)
+		(property "Value" "~"
+			(at 184.15 102.8699 0)
+			(effects
+				(font
+					(size 1.27 1.27)
+				)
+				(justify left)
+			)
+		)
+		(property "Footprint" "modules_footprints:minimal_ad74416h"
+			(at 182.88 109.22 0)
+			(effects
+				(font
+					(size 1.27 1.27)
+				)
+				(justify left)
+				(hide yes)
+			)
+		)
+		(property "Datasheet" ""
+			(at 177.8 101.6 0)
+			(effects
+				(font
+					(size 1.27 1.27)
+				)
+				(hide yes)
+			)
+		)
+		(property "Description" ""
+			(at 177.8 101.6 0)
+			(effects
+				(font
+					(size 1.27 1.27)
+				)
+				(hide yes)
+			)
+		)
+		(instances
+			(project ""
+				(path "/947a17bd-6931-4ad8-bf27-70104debc844"
+					(reference "U1")
+					(unit 1)
+				)
+			)
+		)
+	)
 	(symbol
 		(lib_id "UNITED_MODULES_DATA_BASE:AD74416H_POWER_INTERFACE_MODULE")

Commit message: backup
Parts:
- added U2, U3, U4: ~, modules_footprints:minimal_ad74416h, symbol UNITED_MODULES_DATA_BASE:MINIMAL_AD74416H
Other:
- moved on the sheet: MOD1, U1
Changed lines of the file:
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@@
+	(symbol
+		(lib_id "UNITED_MODULES_DATA_BASE:MINIMAL_AD74416H")
+		(at 160.02 101.6 0)
+		(unit 1)
+		(exclude_from_sim no)
+		(in_bom yes)
+		(on_board yes)
+		(dnp no)
+		(fields_autoplaced yes)
+		(property "Reference" "U1"
+			(at 166.37 100.3299 0)
+			(effects
+				(font
+					(size 1.27 1.27)
+				)
+				(justify left)
+			)
+		)
+		(property "Value" "~"
+			(at 166.37 102.8699 0)
+			(effects
+				(font
+					(size 1.27 1.27)
+				)
+				(justify left)
+			)
+		)
+		(property "Footprint" "modules_footprints:minimal_ad74416h"
+			(at 165.1 109.22 0)
+			(effects
+				(font
+					(size 1.27 1.27)
+				)
+				(justify left)
+				(hide yes)
+			)
+		)
+		(property "Datasheet" ""
+			(at 160.02 101.6 0)
+			(effects
+				(font
+					(size 1.27 1.27)
+				)
+				(hide yes)
+			)
+		)
+		(property "Description" ""
+			(at 160.02 101.6 0)
+			(effects
+				(font
+					(size 1.27 1.27)
+				)
+				(hide yes)
+			)
+		)
+		(instances
+			(project ""
+				(path "/947a17bd-6931-4ad8-bf27-70104debc844"
+					(reference "U1")
+					(unit 1)
+				)
+			)
+		)
+	)
+	(symbol
+		(lib_id "UNITED_MODULES_DATA_BASE:AD74416H_POWER_INTERFACE_MODULE")
+		(at 142.24 101.6 0)
+		(unit 1)
+		(exclude_from_sim no)
+		(in_bom yes)
+		(on_board yes)
+		(dnp no)
+		(fields_autoplaced yes)
+		(property "Reference" "MOD1"
+			(at 148.59 100.3299 0)
+			(effects
+				(font
+					(size 1.27 1.27)
+				)
+				(justify left)
+			)
+		)
+		(property "Value" "~"
+			(at 148.59 102.8699 0)
+			(effects
+				(font
+					(size 1.27 1.27)
+				)
+				(justify left)
+			)
+		)
+		(property "Footprint" "modules_footprints:ad74416h_power_interface_module"
+			(at 142.24 109.22 0)
+			(effects
+				(font
+					(size 1.27 1.27)
+				)
+				(justify left)
+				(hide yes)
+			)
+		)
+		(property "Datasheet" ""
+			(at 142.24 101.6 0)
+			(effects
+				(font
+					(size 1.27 1.27)
+				)
+				(hide yes)
+			)
+		)
+		(property "Description" ""
+			(at 142.24 101.6 0)
+			(effects
+				(font
+					(size 1.27 1.27)
+				)
+				(hide yes)
+			)
+		)
+		(instances
+			(project ""
+				(path "/947a17bd-6931-4ad8-bf27-70104debc844"
+					(reference "MOD1")
+					(unit 1)
+				)
+			)
+		)
+	)
+	(symbol
+		(lib_id "UNITED_MODULES_DATA_BASE:MINIMAL_AD74416H")
+		(at 213.36 101.6 0)
+		(unit 1)
+		(exclude_from_sim no)
+		(in_bom yes)
+		(on_board yes)
+		(dnp no)
+		(fields_autoplaced yes)
+		(property "Reference" "U4"
+			(at 219.71 100.3299 0)
+			(effects
+				(font
+					(size 1.27 1.27)
+				)
+				(justify left)
+			)
+		)
+		(property "Value" "~"
+			(at 219.71 102.8699 0)
+			(effects
+				(font
+					(size 1.27 1.27)
+				)
+				(justify left)
+			)
+		)
+		(property "Footprint" "modules_footprints:minimal_ad74416h"
+			(at 218.44 109.22 0)
+			(effects
+				(font
+					(size 1.27 1.27)
+				)
+				(justify left)
+				(hide yes)
+			)
+		)
+		(property "Datasheet" ""
+			(at 213.36 101.6 0)
+			(effects
+				(font
+					(size 1.27 1.27)
+				)
+				(hide yes)
+			)
+		)
+		(property "Description" ""
+			(at 213.36 101.6 0)
+			(effects
+				(font
+					(size 1.27 1.27)
+				)
+				(hide yes)
+			)
+		)
+		(instances
+			(project "modular_ad74416h_plc"
+				(path "/947a17bd-6931-4ad8-bf27-70104debc844"
+					(reference "U4")
+					(unit 1)
+				)
+			)
+		)
+	)
+	(symbol
+		(lib_id "UNITED_MODULES_DATA_BASE:MINIMAL_AD74416H")
+		(at 195.58 101.6 0)
+		(unit 1)
+		(exclude_from_sim no)
+		(in_bom yes)
+		(on_board yes)
+		(dnp no)
+		(fields_autoplaced yes)
+		(property "Reference" "U3"
+			(at 201.93 100.3299 0)
+			(effects
+				(font
+					(size 1.27 1.27)
+				)
+				(justify left)
+			)
+		)
+		(property "Value" "~"
+			(at 201.93 102.8699 0)
+			(effects
+				(font
+					(size 1.27 1.27)
+				)
+				(justify left)
+			)
+		)
+		(property "Footprint" "modules_footprints:minimal_ad74416h"
+			(at 200.66 109.22 0)
+			(effects
+				(font
+					(size 1.27 1.27)
+				)
+				(justify left)
+				(hide yes)
+			)
+		)
+		(property "Datasheet" ""
+			(at 195.58 101.6 0)
+			(effects
+				(font
+					(size 1.27 1.27)
+				)
+				(hide yes)
+			)
+		)
+		(property "Description" ""
+			(at 195.58 101.6 0)
+			(effects
+				(font
+					(size 1.27 1.27)
+				)
+				(hide yes)
+			)
+		)
+		(instances
+			(project "modular_ad74416h_plc"
+				(path "/947a17bd-6931-4ad8-bf27-70104debc844"
+					(reference "U3")
+					(unit 1)
+				)
+			)
+		)
+	)
 	(symbol
 		(lib_id "UNITED_MODULES_DATA_BASE:MINIMAL_AD74416H")
@@
 		(dnp no)
 		(fields_autoplaced yes)
-		(property "Reference" "U1"
+		(property "Reference" "U2"
 			(at 184.15 100.3299 0)
 			(effects
@@
 		)
 		(instances
-			(project ""
-				(path "/947a17bd-6931-4ad8-bf27-70104debc844"
-					(reference "U1")
-					(unit 1)
-				)
-			)
-		)
-	)
-	(symbol
-		(lib_id "UNITED_MODULES_DATA_BASE:AD74416H_POWER_INTERFACE_MODULE")
-		(at 152.4 101.6 0)
-		(unit 1)
-		(exclude_from_sim no)
-		(in_bom yes)
-		(on_board yes)
-		(dnp no)
-		(fields_autoplaced yes)
-		(property "Reference" "MOD1"
-			(at 158.75 100.3299 0)
-			(effects
-				(font
-					(size 1.27 1.27)
-				)
-				(justify left)
-			)
-		)
-		(property "Value" "~"
-			(at 158.75 102.8699 0)
-			(effects
-				(font
-					(size 1.27 1.27)
-				)
-				(justify left)
-			)
-		)
-		(property "Footprint" "modules_footprints:ad74416h_power_interface_module"
-			(at 152.4 109.22 0)
-			(effects
-				(font
-					(size 1.27 1.27)
-				)
-				(justify left)
-				(hide yes)
-			)
-		)
-		(property "Datasheet" ""
-			(at 152.4 101.6 0)
-			(effects
-				(font
-					(size 1.27 1.27)
-				)
-				(hide yes)
-			)
-		)
-		(property "Description" ""
-			(at 152.4 101.6 0)
-			(effects
-				(font
-					(size 1.27 1.27)
-				)
-				(hide yes)
-			)
-		)
-		(instances
-			(project ""
-				(path "/947a17bd-6931-4ad8-bf27-70104debc844"
-					(reference "MOD1")
-					(unit 1)
-				)
+			(project "modular_ad74416h_plc"
+				(path "/947a17bd-6931-4ad8-bf27-70104debc844"
+					(reference "U2")
+					(unit 1)
+				)

Commit message: backup
Parts:
- added MOD2: ~, modules_footprints:minimal_adp1074, symbol UNITED_MODULES_DATA_BASE:MINIMAL_ADP1074
- added U5: ~, modules_footprints:minimal_adpl76030, symbol UNITED_MODULES_DATA_BASE:MINIMAL_ADPL76030
Changed lines of the file:
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@@
+	)
+	(symbol
+		(lib_id "UNITED_MODULES_DATA_BASE:MINIMAL_ADPL76030")
+		(at 213.36 137.16 0)
+		(unit 1)
+		(exclude_from_sim no)
+		(in_bom yes)
+		(on_board yes)
+		(dnp no)
+		(fields_autoplaced yes)
+		(property "Reference" "U5"
+			(at 219.71 135.8899 0)
+			(effects
+				(font
+					(size 1.27 1.27)
+				)
+				(justify left)
+			)
+		)
+		(property "Value" "~"
+			(at 219.71 138.4299 0)
+			(effects
+				(font
+					(size 1.27 1.27)
+				)
+				(justify left)
+			)
+		)
+		(property "Footprint" "modules_footprints:minimal_adpl76030"
+			(at 218.44 144.78 0)
+			(effects
+				(font
+					(size 1.27 1.27)
+				)
+				(justify left)
+				(hide yes)
+			)
+		)
+		(property "Datasheet" ""
+			(at 213.36 137.16 0)
+			(effects
+				(font
+					(size 1.27 1.27)
+				)
+				(hide yes)
+			)
+		)
+		(property "Description" ""
+			(at 213.36 137.16 0)
+			(effects
+				(font
+					(size 1.27 1.27)
+				)
+				(hide yes)
+			)
+		)
+		(instances
+			(project ""
+				(path "/947a17bd-6931-4ad8-bf27-70104debc844"
+					(reference "U5")
+					(unit 1)
+				)
+			)
+		)
 	)
 	(symbol
@@
 					(unit 1)
 				)
+			)
+		)
+	)
+	(symbol
+		(lib_id "UNITED_MODULES_DATA_BASE:MINIMAL_ADP1074")
+		(at 213.36 119.38 0)
+		(unit 1)
+		(exclude_from_sim no)
+		(in_bom yes)
+		(on_board yes)
+		(dnp no)
+		(fields_autoplaced yes)
+		(property "Reference" "MOD2"
+			(at 219.71 118.1099 0)
+			(effects
+				(font
+					(size 1.27 1.27)
+				)
+				(justify left)
+			)
+		)
+		(property "Value" "~"
+			(at 219.71 120.6499 0)
+			(effects
+				(font
+					(size 1.27 1.27)
+				)
+				(justify left)
+			)
+		)
+		(property "Footprint" "modules_footprints:minimal_adp1074"
+			(at 213.36 127 0)
+			(effects
+				(font
+					(size 1.27 1.27)
+				)
+				(justify left)
+				(hide yes)
+			)
+		)
+		(property "Datasheet" ""
+			(at 213.36 119.38 0)
+			(effects
+				(font
+					(size 1.27 1.27)
+				)
+				(hide yes)
+			)
+		)
+		(property "Description" ""
+			(at 213.36 119.38 0)
+			(effects
+				(font
+					(size 1.27 1.27)
+				)
+				(hide yes)
+			)
+		)
+		(instances
+			(project ""
+				(path "/947a17bd-6931-4ad8-bf27-70104debc844"
+					(reference "MOD2")
+					(unit 1)
+				)

Commit message: backup
Parts:
- added U6: ~, modules_footprints:minimal_ad74416h_stack_adapter, symbol UNITED_MODULES_DATA_BASE:MINIMAL_AD74416H_STACK_ADAPTER
Changed lines of the file:
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@@
 	(paper "A4")
+	(symbol
+		(lib_id "UNITED_MODULES_DATA_BASE:MINIMAL_AD74416H_STACK_ADAPTER")
+		(at 195.58 119.38 0)
+		(unit 1)
+		(exclude_from_sim no)
+		(in_bom yes)
+		(on_board yes)
+		(dnp no)
+		(fields_autoplaced yes)
+		(property "Reference" "U6"
+			(at 201.93 118.1099 0)
+			(effects
+				(font
+					(size 1.27 1.27)
+				)
+				(justify left)
+			)
+		)
+		(property "Value" "~"
+			(at 201.93 120.6499 0)
+			(effects
+				(font
+					(size 1.27 1.27)
+				)
+				(justify left)
+			)
+		)
+		(property "Footprint" "modules_footprints:minimal_ad74416h_stack_adapter"
+			(at 200.66 127 0)
+			(effects
+				(font
+					(size 1.27 1.27)
+				)
+				(justify left)
+				(hide yes)
+			)
+		)
+		(property "Datasheet" ""
+			(at 195.58 119.38 0)
+			(effects
+				(font
+					(size 1.27 1.27)
+				)
+				(hide yes)
+			)
+		)
+		(property "Description" ""
+			(at 195.58 119.38 0)
+			(effects
+				(font
+					(size 1.27 1.27)
+				)
+				(hide yes)
+			)
+		)
+		(instances
+			(project ""
+				(path "/947a17bd-6931-4ad8-bf27-70104debc844"
+					(reference "U6")
+					(unit 1)
+				)
+			)
+		)
+	)
 	(symbol
 		(lib_id "UNITED_MODULES_DATA_BASE:MINIMAL_AD74416H")

Commit message: backup
Parts:
- MOD1: footprint modules_footprints:ad74416h_power_interface_module -> modules_footprints:ad74416h_power_interface_module_v2; symbol UNITED_MODULES_DATA_BASE:AD74416H_POWER_INTERFACE_MODULE -> UNITED_MODULES_DATA_BASE:AD74416H_POWER_INTERFACE_MODULE_v2
- MOD2: footprint modules_footprints:minimal_adp1074 -> modules_footprints:minimal_adp1074_v2; symbol UNITED_MODULES_DATA_BASE:MINIMAL_ADP1074 -> UNITED_MODULES_DATA_BASE:MINIMAL_ADP1074_v2
- MOD5: renamed from U5; footprint modules_footprints:minimal_adpl76030 -> modules_footprints:minimal_adpl76030_v2; symbol UNITED_MODULES_DATA_BASE:MINIMAL_ADPL76030 -> UNITED_MODULES_DATA_BASE:MINIMAL_ADPL76030_v2
- MOD6: renamed from U6; footprint modules_footprints:minimal_ad74416h_stack_adapter -> modules_footprints:minimal_ad74416h_stack_adapter_v2; symbol UNITED_MODULES_DATA_BASE:MINIMAL_AD74416H_STACK_ADAPTER -> UNITED_MODULES_DATA_BASE:MINIMAL_AD74416H_STACK_ADAPTER_v2
Changed lines of the file:
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@@
 	(paper "A4")
 	(symbol
-		(lib_id "UNITED_MODULES_DATA_BASE:MINIMAL_AD74416H_STACK_ADAPTER")
+		(lib_id "UNITED_MODULES_DATA_BASE:MINIMAL_AD74416H_STACK_ADAPTER_v2")
 		(at 195.58 119.38 0)
 		(unit 1)
@@
 		(dnp no)
 		(fields_autoplaced yes)
-		(property "Reference" "U6"
+		(property "Reference" "MOD6"
 			(at 201.93 118.1099 0)
 			(effects
@@
 			)
 		)
-		(property "Footprint" "modules_footprints:minimal_ad74416h_stack_adapter"
+		(property "Footprint" "modules_footprints:minimal_ad74416h_stack_adapter_v2"
 			(at 200.66 127 0)
 			(effects
@@
 			(project ""
 				(path "/947a17bd-6931-4ad8-bf27-70104debc844"
-					(reference "U6")
+					(reference "MOD6")
 					(unit 1)
 				)
@@
 	)
 	(symbol
-		(lib_id "UNITED_MODULES_DATA_BASE:MINIMAL_ADPL76030")
+		(lib_id "UNITED_MODULES_DATA_BASE:MINIMAL_ADPL76030_v2")
 		(at 213.36 137.16 0)
 		(unit 1)
@@
 		(dnp no)
 		(fields_autoplaced yes)
-		(property "Reference" "U5"
+		(property "Reference" "MOD5"
 			(at 219.71 135.8899 0)
 			(effects
@@
 			)
 		)
-		(property "Footprint" "modules_footprints:minimal_adpl76030"
+		(property "Footprint" "modules_footprints:minimal_adpl76030_v2"
 			(at 218.44 144.78 0)
 			(effects
@@
 			(project ""
 				(path "/947a17bd-6931-4ad8-bf27-70104debc844"
-					(reference "U5")
-					(unit 1)
-				)
-			)
-		)
-	)
-	(symbol
-		(lib_id "UNITED_MODULES_DATA_BASE:AD74416H_POWER_INTERFACE_MODULE")
+					(reference "MOD5")
+					(unit 1)
+				)
+			)
+		)
+	)
+	(symbol
+		(lib_id "UNITED_MODULES_DATA_BASE:AD74416H_POWER_INTERFACE_MODULE_v2")
 		(at 142.24 101.6 0)
 		(unit 1)
@@
 			)
 		)
-		(property "Footprint" "modules_footprints:ad74416h_power_interface_module"
+		(property "Footprint" "modules_footprints:ad74416h_power_interface_module_v2"
 			(at 142.24 109.22 0)
 			(effects
@@
 	)
 	(symbol
-		(lib_id "UNITED_MODULES_DATA_BASE:MINIMAL_ADP1074")
+		(lib_id "UNITED_MODULES_DATA_BASE:MINIMAL_ADP1074_v2")
 		(at 213.36 119.38 0)
 		(unit 1)
@@
 			)
 		)
-		(property "Footprint" "modules_footprints:minimal_adp1074"
+		(property "Footprint" "modules_footprints:minimal_adp1074_v2"
 			(at 213.36 127 0)
 			(effects

Commit message: backup
Parts:
- added M1: ~, mechanical_parts:2203350, symbol UNITED_MECHANICAL_DATA_BASE:M_2203350
Changed lines of the file:
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@@
+	)
+	(symbol
+		(lib_id "UNITED_MECHANICAL_DATA_BASE:M_2203350")
+		(at 74.93 151.13 0)
+		(unit 1)
+		(exclude_from_sim no)
+		(in_bom yes)
+		(on_board yes)
+		(dnp no)
+		(fields_autoplaced yes)
+		(property "Reference" "M1"
+			(at 88.9 149.8599 0)
+			(effects
+				(font
+					(size 1.27 1.27)
+				)
+				(justify left)
+			)
+		)
+		(property "Value" "~"
+			(at 88.9 152.3999 0)
+			(effects
+				(font
+					(size 1.27 1.27)
+				)
+				(justify left)
+			)
+		)
+		(property "Footprint" "mechanical_parts:2203350"
+			(at 74.93 166.37 0)
+			(effects
+				(font
+					(size 1.27 1.27)
+				)
+				(justify left)
+				(hide yes)
+			)
+		)
+		(property "Datasheet" "https://product-download.phoenixcontact.com/8025199?response-content-disposition=inline;%20filename%3D%22pxc_2203350_00_02_UCS-HH-125-87-9005_2D.pdf%22&Expires=1760989045&Signature=yE5~e9oEp1czmAuNjEVI-zMCk115UdZsJSv~rrHj0mJAaEc55~bR20bW9JJOB3hki3HOREKBknujH~8gYOUKHzLpSGgETtHOQerG8jWvvCgEOtBdmOWxPCFsOz9Wsha5f2~VPSQJvuGHCf2CTsN5w1iZpHUNsgk-mkW2p9pzyOLKxVWYhtjSbQv3gEOsVOjFHlOlmTX7rqb6sJSqriLur8mA9m3Tjg-Z30FHvQ1KxAkSK4hrzVgTKxESnhz77NCWnp-s970KOF79zwJtK4mF8zDCIv5i5t6kHDL5A9xxqz5SxQzMk3O-D3HhNnTfdPWE6WLROkbUQOZ4tbjTyLeyWA__&Key-Pair-Id=K1I2N54A7B0GD"
+			(at 74.93 168.91 0)
+			(effects
+				(font
+					(size 1.27 1.27)
+				)
+				(justify left)
+				(hide yes)
+			)
+		)
+		(property "Description" "UCS HH 125-87 9005 - Housing half shell"
+			(at 74.93 171.45 0)
+			(effects
+				(font
+					(size 1.27 1.27)
+				)
+				(justify left)
+				(hide yes)
+			)
+		)
+		(instances
+			(project ""
+				(path "/947a17bd-6931-4ad8-bf27-70104debc844"
+					(reference "M1")
+					(unit 1)
+				)
+			)
+		)
 	)
 	(symbol

Commit message: backup
Parts:
- added M2, M3, M4, M5: ~, mechanical_parts:2203404_v2, symbol UNITED_MECHANICAL_DATA_BASE:M_2203404_v2
Other:
- moved on the sheet: M1
