File: modular_ad74416h_plc/modular_ad74416h_plc.kicad_sch (KiCad schematic)
At the start: 13 parts

Commit message: backup
Parts:
- added M6, M7, M8, M9: ~, mechanical_parts:2203400, symbol UNITED_MECHANICAL_DATA_BASE:M_2203400

Commit message: backup
Parts:
- added M10: ~, mechanical_parts:2203350, symbol UNITED_MECHANICAL_DATA_BASE:M_2203350
Changed lines of the file:
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@@
+	)
+	(symbol
+		(lib_id "UNITED_MECHANICAL_DATA_BASE:M_2203350")
+		(at 76.2 182.88 0)
+		(unit 1)
+		(exclude_from_sim no)
+		(in_bom yes)
+		(on_board yes)
+		(dnp no)
+		(fields_autoplaced yes)
+		(property "Reference" "M10"
+			(at 90.17 181.6099 0)
+			(effects
+				(font
+					(size 1.27 1.27)
+				)
+				(justify left)
+			)
+		)
+		(property "Value" "~"
+			(at 90.17 184.1499 0)
+			(effects
+				(font
+					(size 1.27 1.27)
+				)
+				(justify left)
+			)
+		)
+		(property "Footprint" "mechanical_parts:2203350"
+			(at 76.2 198.12 0)
+			(effects
+				(font
+					(size 1.27 1.27)
+				)
+				(justify left)
+				(hide yes)
+			)
+		)
+		(property "Datasheet" "https://product-download.phoenixcontact.com/8025199?response-content-disposition=inline;%20filename%3D%22pxc_2203350_00_02_UCS-HH-125-87-9005_2D.pdf%22&Expires=1760989045&Signature=yE5~e9oEp1czmAuNjEVI-zMCk115UdZsJSv~rrHj0mJAaEc55~bR20bW9JJOB3hki3HOREKBknujH~8gYOUKHzLpSGgETtHOQerG8jWvvCgEOtBdmOWxPCFsOz9Wsha5f2~VPSQJvuGHCf2CTsN5w1iZpHUNsgk-mkW2p9pzyOLKxVWYhtjSbQv3gEOsVOjFHlOlmTX7rqb6sJSqriLur8mA9m3Tjg-Z30FHvQ1KxAkSK4hrzVgTKxESnhz77NCWnp-s970KOF79zwJtK4mF8zDCIv5i5t6kHDL5A9xxqz5SxQzMk3O-D3HhNnTfdPWE6WLROkbUQOZ4tbjTyLeyWA__&Key-Pair-Id=K1I2N54A7B0GD"
+			(at 76.2 200.66 0)
+			(effects
+				(font
+					(size 1.27 1.27)
+				)
+				(justify left)
+				(hide yes)
+			)
+		)
+		(property "Description" "UCS HH 125-87 9005 - Housing half shell"
+			(at 76.2 203.2 0)
+			(effects
+				(font
+					(size 1.27 1.27)
+				)
+				(justify left)
+				(hide yes)
+			)
+		)
+		(instances
+			(project "modular_ad74416h_plc"
+				(path "/947a17bd-6931-4ad8-bf27-70104debc844"
+					(reference "M10")
+					(unit 1)
+				)
+			)
+		)
 	)
 	(symbol

Commit message: backup
Parts:
- added M11, M12: ~, mechanical_parts:2203362, symbol UNITED_MECHANICAL_DATA_BASE:M_2203362
- added M13, M14: ~, mechanical_parts:2203369, symbol UNITED_MECHANICAL_DATA_BASE:M_2203369
Other:
- moved on the sheet: M1, M10, M2, M3, M4, M5, M6, M7, M8, M9

Commit message: backup
Parts:
- M11: footprint mechanical_parts:2203362 -> mechanical_parts:2203362_v3; symbol UNITED_MECHANICAL_DATA_BASE:M_2203362 -> UNITED_MECHANICAL_DATA_BASE:M_2203362_v3
- M12: footprint mechanical_parts:2203362 -> mechanical_parts:2203362_v2; symbol UNITED_MECHANICAL_DATA_BASE:M_2203362 -> UNITED_MECHANICAL_DATA_BASE:M_2203362_v2
- M13: footprint mechanical_parts:2203369 -> mechanical_parts:2203369_v2; symbol UNITED_MECHANICAL_DATA_BASE:M_2203369 -> UNITED_MECHANICAL_DATA_BASE:M_2203369_v2
- M14: footprint mechanical_parts:2203369 -> mechanical_parts:2203369_v3; symbol UNITED_MECHANICAL_DATA_BASE:M_2203369 -> UNITED_MECHANICAL_DATA_BASE:M_2203369_v3
Changed lines of the file:
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@@
 	)
 	(symbol
-		(lib_id "UNITED_MECHANICAL_DATA_BASE:M_2203362")
+		(lib_id "UNITED_MECHANICAL_DATA_BASE:M_2203362_v2")
 		(at 76.2 78.74 0)
 		(unit 1)
@@
 			)
 		)
-		(property "Footprint" "mechanical_parts:2203362"
+		(property "Footprint" "mechanical_parts:2203362_v2"
 			(at 76.2 81.28 0)
 			(effects
@@
 	)
 	(symbol
-		(lib_id "UNITED_MECHANICAL_DATA_BASE:M_2203362")
+		(lib_id "UNITED_MECHANICAL_DATA_BASE:M_2203362_v3")
 		(at 76.2 124.46 0)
 		(unit 1)
@@
 			)
 		)
-		(property "Footprint" "mechanical_parts:2203362"
+		(property "Footprint" "mechanical_parts:2203362_v3"
 			(at 76.2 127 0)
 			(effects
@@
 	)
 	(symbol
-		(lib_id "UNITED_MECHANICAL_DATA_BASE:M_2203369")
+		(lib_id "UNITED_MECHANICAL_DATA_BASE:M_2203369_v2")
 		(at 99.06 101.6 270)
 		(unit 1)
@@
 			)
 		)
-		(property "Footprint" "mechanical_parts:2203369"
+		(property "Footprint" "mechanical_parts:2203369_v2"
 			(at 96.52 101.6 0)
 			(effects
@@
 	)
 	(symbol
-		(lib_id "UNITED_MECHANICAL_DATA_BASE:M_2203369")
+		(lib_id "UNITED_MECHANICAL_DATA_BASE:M_2203369_v3")
 		(at 53.34 101.6 90)
 		(mirror x)
@@
 		(dnp no)
 		(property "Reference" "M14"
-			(at 50.8 100.3299 90)
-			(effects
-				(font
-					(size 1.27 1.27)
-				)
-				(justify left)
-			)
-		)
-		(property "Value" "~"
-			(at 50.8 102.8699 90)
-			(effects
-				(font
-					(size 1.27 1.27)
-				)
-				(justify left)
-			)
-		)
-		(property "Footprint" "mechanical_parts:2203369"
+			(at 50.8 101.6 0)
+			(effects
+				(font
+					(size 1.27 1.27)
+				)
+				(justify left)
+			)
+		)
+		(property "Value" "~"
+			(at 53.34 101.6 0)
+			(effects
+				(font
+					(size 1.27 1.27)
+				)
+				(justify left)
+			)
+		)
+		(property "Footprint" "mechanical_parts:2203369_v3"
 			(at 55.88 101.6 0)
 			(effects

Commit message: backup
Parts:
- M11: footprint mechanical_parts:2203362_v3 -> mechanical_parts:2203362_v2; symbol UNITED_MECHANICAL_DATA_BASE:M_2203362_v3 -> UNITED_MECHANICAL_DATA_BASE:M_2203362_v2
- M14: footprint mechanical_parts:2203369_v3 -> mechanical_parts:2203369_v2; symbol UNITED_MECHANICAL_DATA_BASE:M_2203369_v3 -> UNITED_MECHANICAL_DATA_BASE:M_2203369_v2
Changed lines of the file:
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@@
 	)
 	(symbol
-		(lib_id "UNITED_MECHANICAL_DATA_BASE:M_2203362_v3")
+		(lib_id "UNITED_MECHANICAL_DATA_BASE:M_2203362_v2")
 		(at 76.2 124.46 0)
 		(unit 1)
@@
 			)
 		)
-		(property "Footprint" "mechanical_parts:2203362_v3"
+		(property "Footprint" "mechanical_parts:2203362_v2"
 			(at 76.2 127 0)
 			(effects
@@
 	)
 	(symbol
-		(lib_id "UNITED_MECHANICAL_DATA_BASE:M_2203369_v3")
+		(lib_id "UNITED_MECHANICAL_DATA_BASE:M_2203369_v2")
 		(at 53.34 101.6 90)
 		(mirror x)
@@
 			)
 		)
-		(property "Footprint" "mechanical_parts:2203369_v3"
+		(property "Footprint" "mechanical_parts:2203369_v2"
 			(at 55.88 101.6 0)
 			(effects
