File: modular_ad74416h_plc/modular_ad74416h_plc.kicad_sch (KiCad schematic)
At the start: 22 parts

Commit message: Sync changes to both main and doc_workflow branches
Parts:
- renumbered U1 to A1, U2 to A2, U3 to A3, U4 to A4
Changed lines of the file:
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@@
 	)
 	(symbol
+		(lib_name "MINIMAL_AD74416H_1")
 		(lib_id "UNITED_MODULES_DATA_BASE:MINIMAL_AD74416H")
 		(at 160.02 101.6 0)
@@
 		(dnp no)
 		(fields_autoplaced yes)
-		(property "Reference" "U1"
+		(property "Reference" "A1"
 			(at 166.37 100.3299 0)
 			(effects
@@
 			(project ""
 				(path "/947a17bd-6931-4ad8-bf27-70104debc844"
-					(reference "U1")
+					(reference "A1")
 					(unit 1)
 				)
@@
 		(dnp no)
 		(fields_autoplaced yes)
-		(property "Reference" "U4"
+		(property "Reference" "A4"
 			(at 219.71 100.3299 0)
 			(effects
@@
 			(project "modular_ad74416h_plc"
 				(path "/947a17bd-6931-4ad8-bf27-70104debc844"
-					(reference "U4")
-					(unit 1)
-				)
-			)
-		)
-	)
-	(symbol
+					(reference "A4")
+					(unit 1)
+				)
+			)
+		)
+	)
+	(symbol
+		(lib_name "MINIMAL_AD74416H_3")
 		(lib_id "UNITED_MODULES_DATA_BASE:MINIMAL_AD74416H")
 		(at 195.58 101.6 0)
@@
 		(dnp no)
 		(fields_autoplaced yes)
-		(property "Reference" "U3"
+		(property "Reference" "A3"
 			(at 201.93 100.3299 0)
 			(effects
@@
 			(project "modular_ad74416h_plc"
 				(path "/947a17bd-6931-4ad8-bf27-70104debc844"
-					(reference "U3")
+					(reference "A3")
 					(unit 1)
 				)
@@
 	)
 	(symbol
+		(lib_name "MINIMAL_AD74416H_2")
 		(lib_id "UNITED_MODULES_DATA_BASE:MINIMAL_AD74416H")
 		(at 177.8 101.6 0)
@@
 		(dnp no)
 		(fields_autoplaced yes)
-		(property "Reference" "U2"
+		(property "Reference" "A2"
 			(at 184.15 100.3299 0)
 			(effects
@@
 			(project "modular_ad74416h_plc"
 				(path "/947a17bd-6931-4ad8-bf27-70104debc844"
-					(reference "U2")
-					(unit 1)
-				)
+					(reference "A2")
+					(unit 1)
+				)

Commit message: backup
Parts:
- renumbered MOD6 to A6
Changed lines of the file:
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@@
 		(dnp no)
 		(fields_autoplaced yes)
-		(property "Reference" "MOD6"
+		(property "Reference" "A6"
 			(at 201.93 118.1099 0)
 			(effects
@@
 			(project ""
 				(path "/947a17bd-6931-4ad8-bf27-70104debc844"
-					(reference "MOD6")
+					(reference "A6")
 					(unit 1)
 				)

Commit message: backup
Parts:
- renumbered MOD1 to A5, MOD5 to A7
Changed lines of the file:
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@@
 		(dnp no)
 		(fields_autoplaced yes)
-		(property "Reference" "MOD5"
+		(property "Reference" "A7"
 			(at 219.71 135.8899 0)
 			(effects
@@
 			(project ""
 				(path "/947a17bd-6931-4ad8-bf27-70104debc844"
-					(reference "MOD5")
+					(reference "A7")
 					(unit 1)
 				)
@@
 		(dnp no)
 		(fields_autoplaced yes)
-		(property "Reference" "MOD1"
+		(property "Reference" "A5"
 			(at 148.59 100.3299 0)
 			(effects
@@
 			(project ""
 				(path "/947a17bd-6931-4ad8-bf27-70104debc844"
-					(reference "MOD1")
+					(reference "A5")
 					(unit 1)
 				)

Commit message: backup
Parts:
- renumbered MOD2 to A8
Changed lines of the file:
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@@
 		(dnp no)
 		(fields_autoplaced yes)
-		(property "Reference" "MOD2"
+		(property "Reference" "A8"
 			(at 219.71 118.1099 0)
 			(effects
@@
 			(project ""
 				(path "/947a17bd-6931-4ad8-bf27-70104debc844"
-					(reference "MOD2")
+					(reference "A8")
 					(unit 1)
 				)
